Commit message: Added EZGripper as end effector

File: manipulator_h_description/urdf/manipulator_h.xacro (robot description, xacro)
@@ -2,293 +2,443 @@
 <!-- Revolute-Revolute Manipulator -->
 <robot name="robotis_manipulator_h" xmlns:xacro="http://www.ros.org/wiki/xacro">
-  <!-- some parameters -->
-  <xacro:property name="pi" value="3.141592654" />
-  <!-- some parameters -->
-  <xacro:property name="pi" value="3.141592654" />
-  <!-- Import all Gazebo-customization elements, including Gazebo colors -->
-  <xacro:include filename="$(find manipulator_h_description)/urdf/manipulator_h.gazebo" />
-  <!-- Import Rviz colors -->
-  <xacro:include filename="$(find manipulator_h_description)/urdf/materials.xacro" />
-  <!-- Used for fixing robot to Gazebo 'link 1' -->
-  <link name="world">
-  </link>
-  <joint name="world_fixed" type="fixed">
-    <origin xyz="0 0 0" rpy="0 0 0"/>
-    <parent link="world"/>
-    <child link="link1"/>
-  </joint>
-  <!-- link 1 -->
-  <link name="link1">
-    <collision>
-      <origin xyz="0 0 0" rpy="0 0 0"/>
-      <geometry>
-        <mesh filename="package://manipulator_h_description/meshes/link_1.stl" scale="0.001 0.001 0.001"/>
-      </geometry>
-    </collision>
-    <visual>
-      <origin xyz="0 0 0" rpy="0 0 0"/>
-      <geometry>
-        <mesh filename="package://manipulator_h_description/meshes/link_1.stl" scale="0.001 0.001 0.001"/>
-      </geometry>
-      <material name="grey"/>
-    </visual>
-    <inertial>
-      <origin xyz="0.00023 0.00000 0.06223" rpy="0 0 0"/>
-      <!--<origin xyz="0.00023 0.00000 -0.06377" rpy="0 0 0"/>-->
-      <mass value="0.85644"/>
-      <inertia ixx="1.0" ixy="0.0" ixz="0.0" iyy="1.0" iyz="0.0" izz="1.0" />
-      <!--<inertia ixx="0.00121064" ixy="0.0" ixz="0.00001100" iyy="0.00120886" iyz="0.0" izz="0.00038103" />-->
-    </inertial>
-  </link>
-  <!-- Joint 1 -->
-  <joint name="joint1" type="revolute">
-    <parent link="link1"/>
-    <child link="link2"/>
-    <origin xyz="0.0 0.0 0.126" rpy="0 0 0"/>
-    <axis xyz="0 0 1"/>
-    <limit velocity="6.5" effort="1000" lower="${-pi*0.5}" upper="${pi*0.5}" />
-    <dynamics damping="0.7"/>
-  </joint>
-  <transmission name="tran1">
-    <type>transmission_interface/SimpleTransmission</type>
-    <joint name="joint1">
-      <hardwareInterface>EffortJointInterface</hardwareInterface>
-    </joint>
-    <actuator name="motor1">
-      <hardwareInterface>EffortJointInterface</hardwareInterface>
-      <mechanicalReduction>1</mechanicalReduction>
-    </actuator>
-  </transmission>
-  <!-- link 2 -->
-  <link name="link2">
-    <collision>
-      <origin xyz="0 0 0" rpy="0 0 0"/>
-      <geometry>
-        <mesh filename="package://manipulator_h_description/meshes/link_2.stl" scale="0.001 0.001 0.001"/>
-      </geometry>
-    </collision>
-    <visual>
-      <origin xyz="0 0 0" rpy="0 0 0"/>
-      <geometry>
-        <mesh filename="package://manipulator_h_description/meshes/link_2.stl" scale="0.001 0.001 0.001"/>
-      </geometry>
-      <material name="grey"/>
-    </visual>
-    <inertial>
-      <origin xyz="0.00000 0.00080 0.03183" rpy="0 0 0"/>
-      <!--<origin xyz="0.00000 -0.06820 -0.00117" rpy="0 0 0"/>-->
-      <mass value="0.94658"/>
-      <inertia ixx="1.0" ixy="0.0" ixz="0.0" iyy="1.0" iyz="0.0" izz="1.0" />
-      <!--<inertia ixx="0.00152547" ixy="0.0" ixz="0.0" iyy="0.00045954" iyz="-0.00001086" izz="0.00151740" />-->
-    </inertial>
-  </link>
-  <!-- Joint 2 -->
-  <joint name="joint2" type="revolute">
-    <parent link="link2"/>
-    <child link="link3"/>
-    <origin xyz="0.0 0.069 0.033" rpy="0 0 0"/>
-    <axis xyz="0 1 0"/>
-    <limit velocity="6.5" effort="1000" lower="${-pi*0.5}" upper="${pi*0.5}" />
-    <dynamics damping="0.7"/>
-  </joint>
-  <transmission name="tran2">
-    <type>transmission_interface/SimpleTransmission</type>
-    <joint name="joint2">
-      <hardwareInterface>EffortJointInterface</hardwareInterface>
-    </joint>
-    <actuator name="motor2">
-      <hardwareInterface>EffortJointInterface</hardwareInterface>
-      <mechanicalReduction>1</mechanicalReduction>
-    </actuator>
-  </transmission>
-  <!-- link 3 -->
-  <link name="link3">
-    <collision>
-      <origin xyz="0 0 0" rpy="0 0 0"/>
-      <geometry>
-        <mesh filename="package://manipulator_h_description/meshes/link_3.stl" scale="0.001 0.001 0.001"/>
-      </geometry>
-    </collision>
-    <visual>
-      <origin xyz="0 0 0" rpy="0 0 0"/>
-      <geometry>
-        <mesh filename="package://manipulator_h_description/meshes/link_3.stl" scale="0.001 0.001 0.001"/>
-      </geometry>
-      <material name="grey"/>
-    </visual>
-    <inertial>
-      <origin xyz="0.01768 -0.06881 0.20524" rpy="0 0 0"/>
-      <!--<origin xyz="-0.01232 -0.05731 -0.05876" rpy="0 0 0"/>-->
-      <mass value="1.30260"/>
-      <inertia ixx="1.0" ixy="0.0" ixz="0.0" iyy="1.0" iyz="0.0" izz="1.0" />
-      <!--<inertia ixx="0.01111021" ixy="0.00001331" ixz="-0.00134208" iyy="0.01046642" iyz="0.00016235" izz="0.00202081" />-->
-    </inertial>
-  </link>
-  <!-- Joint 3 -->
-  <joint name="joint3" type="revolute">
-    <parent link="link3"/>
-    <child link="link4"/>
-    <origin xyz="0.03000 -0.01150 0.26400" rpy="0 0 0"/>
-    <axis xyz="0 1 0"/>
-    <limit velocity="6.5" effort="1000" lower="${-pi*0.5}" upper="${pi*0.5}" />
-    <dynamics damping="0.7"/>
-  </joint>
-  <transmission name="tran3">
-    <type>transmission_interface/SimpleTransmission</type>
-    <joint name="joint3">
-      <hardwareInterface>EffortJointInterface</hardwareInterface>
-    </joint>
-    <actuator name="motor3">
-      <hardwareInterface>EffortJointInterface</hardwareInterface>
-      <mechanicalReduction>1</mechanicalReduction>
-    </actuator>
-  </transmission>
-  <!-- link 4 -->
-  <link name="link4">
-    <collision>
-      <origin xyz="0 0 0" rpy="0 0 0"/>
-      <geometry>
-        <mesh filename="package://manipulator_h_description/meshes/link_4.stl" scale="0.001 0.001 0.001"/>
-      </geometry>
-    </collision>
-    <visual>
-      <origin xyz="0 0 0" rpy="0 0 0"/>
-      <geometry>
-        <mesh filename="package://manipulator_h_description/meshes/link_4.stl" scale="0.001 0.001 0.001"/>
-      </geometry>
-      <material name="grey"/>
-    </visual>
-    <inertial>
-      <origin xyz="0.12475 -0.05716 0.02979" rpy="0 0 0"/>
-      <!--<origin xyz="-0.07025 0.00034 -0.00021" rpy="0 0 0"/>-->
-      <mass value="1.15977"/>
-      <inertia ixx="1.0" ixy="0.0" ixz="0.0" iyy="1.0" iyz="0.0" izz="1.0" />
-      <!--<inertia ixx="0.00096726" ixy="0.00004383" ixz="-0.00002771" iyy="0.00318801" iyz="0.00000627" izz="0.00341484" />-->
-    </inertial>
-  </link>
-  <!-- Joint 4 -->
-  <joint name="joint4" type="revolute">
-    <parent link="link4"/>
-    <child link="link5"/>
-    <origin xyz="0.19500 -0.05750 0.03000" rpy="0 0 0"/>
-    <axis xyz="1 0 0"/>
-    <limit velocity="6.5" effort="1000" lower="${-pi*0.5}" upper="${pi*0.5}" />
-    <dynamics damping="0.7"/>
-  </joint>
-  <transmission name="tran4">
-    <type>transmission_interface/SimpleTransmission</type>
-    <joint name="joint4">
-      <hardwareInterface>EffortJointInterface</hardwareInterface>
-    </joint>
-    <actuator name="motor4">
-      <hardwareInterface>EffortJointInterface</hardwareInterface>
-      <mechanicalReduction>1</mechanicalReduction>
-    </actuator>
-  </transmission>
-  <!-- link 5 -->
-  <link name="link5">
-    <collision>
-      <origin xyz="0 0 0" rpy="0 0 0"/>
-      <geometry>
-        <mesh filename="package://manipulator_h_description/meshes/link_5.stl" scale="0.001 0.001 0.001"/>
-      </geometry>
-    </collision>
-    <visual>
-      <origin xyz="0 0 0" rpy="0 0 0"/>
-      <geometry>
-        <mesh filename="package://manipulator_h_description/meshes/link_5.stl" scale="0.001 0.001 0.001"/>
-      </geometry>
-      <material name="grey"/>
-    </visual>
-    <inertial>
-      <origin xyz="0.05642 -0.00217 0.00002" rpy="0 0 0"/>
-      <!--<origin xyz="-0.00658 -0.04717 0.00002" rpy="0 0 0"/>-->
-      <mass value="0.44688"/>
-      <inertia ixx="1.0" ixy="0.0" ixz="0.0" iyy="1.0" iyz="0.0" izz="1.0" />
-      <!--<inertia ixx="0.00030285" ixy="0.00000761" ixz="0.00000031" iyy="0.00022339" iyz="-0.00000001" izz="0.00039766" />-->
-    </inertial>
-  </link>
-  <!-- Joint 5 -->
-  <joint name="joint5" type="revolute">
-    <parent link="link5"/>
-    <child link="link6"/>
-    <origin xyz="0.06300 0.04500 0.00000" rpy="0 0 0"/>
-    <axis xyz="0 1 0"/>
-    <limit velocity="6.5" effort="1000" lower="${-pi*0.5}" upper="${pi*0.5}" />
-    <dynamics damping="0.7"/>
-  </joint>
-  <transmission name="tran5">
-    <type>transmission_interface/SimpleTransmission</type>
-    <joint name="joint5">
-      <hardwareInterface>EffortJointInterface</hardwareInterface>
-    </joint>
-    <actuator name="motor5">
-      <hardwareInterface>EffortJointInterface</hardwareInterface>
-      <mechanicalReduction>1</mechanicalReduction>
-    </actuator>
-  </transmission>
-  <!-- link 6 -->
-  <link name="link6">
-    <collision>
-      <origin xyz="0 0 0" rpy="0 0 0"/>
-      <geometry>
-        <mesh filename="package://manipulator_h_description/meshes/link_6.stl" scale="0.001 0.001 0.001"/>
-      </geometry>
-    </collision>
-    <visual>
-      <origin xyz="0 0 0" rpy="0 0 0"/>
-      <geometry>
-        <mesh filename="package://manipulator_h_description/meshes/link_6.stl" scale="0.001 0.001 0.001"/>
-      </geometry>
-      <material name="grey"/>
-    </visual>
-    <inertial>
-      <origin xyz="0.06831 -0.04457 0.00000" rpy="0 0 0"/>
-      <!--<origin xyz="-0.05469 0.00043 0.00000" rpy="0 0 0"/>-->
-      <mass value="0.43273"/>
-      <inertia ixx="1.0" ixy="0.0" ixz="0.0" iyy="1.0" iyz="0.0" izz="1.0" />
-      <!--<inertia ixx="0.00021512" ixy="0.00001009" ixz="0.00000000" iyy="0.00042827" iyz="0.00000000" izz="0.00051436" />-->
-    </inertial>
-  </link>
-  <!-- Joint 6 -->
-  <joint name="joint6" type="revolute">
-    <parent link="link6"/>
-    <child link="end_link"/>
-    <origin xyz="0.12300 -0.04500 0.00000" rpy="0 0 0"/>
-    <axis xyz="1 0 0"/>
-    <limit velocity="6.5" effort="1000" lower="${-pi*0.5}" upper="${pi*0.5}" />
-    <dynamics damping="0.7"/>
-  </joint>
-  <transmission name="tran6">
-    <type>transmission_interface/SimpleTransmission</type>
-    <joint name="joint6">
-      <hardwareInterface>EffortJointInterface</hardwareInterface>
-    </joint>
-    <actuator name="motor6">
-      <hardwareInterface>EffortJointInterface</hardwareInterface>
-      <mechanicalReduction>1</mechanicalReduction>
-    </actuator>
-  </transmission>
-  <!-- end link -->
-  <link name="end_link">
-    <collision>
-      <origin xyz="0 0 0" rpy="0 0 0"/>
-      <geometry>
-        <mesh filename="package://manipulator_h_description/meshes/end_link.stl" scale="0.001 0.001 0.001"/>
-      </geometry>
-    </collision>
-    <visual>
-      <origin xyz="0 0 0" rpy="0 0 0"/>
-      <geometry>
-        <mesh filename="package://manipulator_h_description/meshes/end_link.stl" scale="0.001 0.001 0.001"/>
-      </geometry>
-      <material name="grey"/>
-    </visual>
-    <inertial>
-      <origin xyz="0.00337 0.00000 0.00000" rpy="0 0 0"/>
-      <mass value="0.01919"/>
-      <inertia ixx="1.0" ixy="0.0" ixz="0.0" iyy="1.0" iyz="0.0" izz="1.0" />
-      <!--<inertia ixx="0.00000938" ixy="0.0" ixz="0.0" iyy="0.00000338" iyz="0.0" izz="0.00000635" />-->
-    </inertial>
-  </link>
+    <!-- some parameters -->
+    <xacro:property name="pi" value="3.141592654" />
+    <!-- some parameters -->
+    <xacro:property name="pi" value="3.141592654" />
+    <!-- Import all Gazebo-customization elements, including Gazebo colors -->
+    <xacro:include filename="$(find manipulator_h_description)/urdf/manipulator_h.gazebo" />
+    <!-- Import Rviz colors -->
+    <xacro:include filename="$(find manipulator_h_description)/urdf/materials.xacro" />
+    <!-- Used for fixing robot to Gazebo 'link 1' -->
+    <link name="world">
+    </link>
+    <joint name="world_fixed" type="fixed">
+        <origin xyz="0 0 0" rpy="0 0 0"/>
+        <parent link="world"/>
+        <child link="link1"/>
+    </joint>
+    <!-- link 1 -->
+    <link name="link1">
+        <collision>
+            <origin xyz="0 0 0" rpy="0 0 0"/>
+            <geometry>
+                <mesh filename="package://manipulator_h_description/meshes/link_1.stl" scale="0.001 0.001 0.001"/>
+            </geometry>
+        </collision>
+        <visual>
+            <origin xyz="0 0 0" rpy="0 0 0"/>
+            <geometry>
+                <mesh filename="package://manipulator_h_description/meshes/link_1.stl" scale="0.001 0.001 0.001"/>
+            </geometry>
+            <material name="grey"/>
+        </visual>
+        <inertial>
+            <origin xyz="0.00023 0.00000 0.06223" rpy="0 0 0"/>
+            <!--<origin xyz="0.00023 0.00000 -0.06377" rpy="0 0 0"/>-->
+            <mass value="0.85644"/>
+            <inertia ixx="1.0" ixy="0.0" ixz="0.0" iyy="1.0" iyz="0.0" izz="1.0" />
+            <!--<inertia ixx="0.00121064" ixy="0.0" ixz="0.00001100" iyy="0.00120886" iyz="0.0" izz="0.00038103" />-->
+        </inertial>
+    </link>
+    <!-- Joint 1 -->
+    <joint name="joint1" type="revolute">
+        <parent link="link1"/>
+        <child link="link2"/>
+        <origin xyz="0.0 0.0 0.126" rpy="0 0 0"/>
+        <axis xyz="0 0 1"/>
+        <limit velocity="6.5" effort="1000" lower="${-pi*0.5}" upper="${pi*0.5}" />
+        <dynamics damping="0.7"/>
+    </joint>
+    <transmission name="tran1">
+        <type>transmission_interface/SimpleTransmission</type>
+        <joint name="joint1">
+            <hardwareInterface>EffortJointInterface</hardwareInterface>
+        </joint>
+        <actuator name="motor1">
+            <hardwareInterface>EffortJointInterface</hardwareInterface>
+            <mechanicalReduction>1</mechanicalReduction>
+        </actuator>
+    </transmission>
+    <!-- link 2 -->
+    <link name="link2">
+        <collision>
+            <origin xyz="0 0 0" rpy="0 0 0"/>
+            <geometry>
+                <mesh filename="package://manipulator_h_description/meshes/link_2.stl" scale="0.001 0.001 0.001"/>
+            </geometry>
+        </collision>
+        <visual>
+            <origin xyz="0 0 0" rpy="0 0 0"/>
+            <geometry>
+                <mesh filename="package://manipulator_h_description/meshes/link_2.stl" scale="0.001 0.001 0.001"/>
+            </geometry>
+            <material name="grey"/>
+        </visual>
+        <inertial>
+            <origin xyz="0.00000 0.00080 0.03183" rpy="0 0 0"/>
+            <!--<origin xyz="0.00000 -0.06820 -0.00117" rpy="0 0 0"/>-->
+            <mass value="0.94658"/>
+            <inertia ixx="1.0" ixy="0.0" ixz="0.0" iyy="1.0" iyz="0.0" izz="1.0" />
+            <!--<inertia ixx="0.00152547" ixy="0.0" ixz="0.0" iyy="0.00045954" iyz="-0.00001086" izz="0.00151740" />-->
+        </inertial>
+    </link>
+    <!-- Joint 2 -->
+    <joint name="joint2" type="revolute">
+        <parent link="link2"/>
+        <child link="link3"/>
+        <origin xyz="0.0 0.069 0.033" rpy="0 0 0"/>
+        <axis xyz="0 1 0"/>
+        <limit velocity="6.5" effort="1000" lower="${-pi*0.5}" upper="${pi*0.5}" />
+        <dynamics damping="0.7"/>
+    </joint>
+    <transmission name="tran2">
+        <type>transmission_interface/SimpleTransmission</type>
+        <joint name="joint2">
+            <hardwareInterface>EffortJointInterface</hardwareInterface>
+        </joint>
+        <actuator name="motor2">
+            <hardwareInterface>EffortJointInterface</hardwareInterface>
+            <mechanicalReduction>1</mechanicalReduction>
+        </actuator>
+    </transmission>
+    <!-- link 3 -->
+    <link name="link3">
+        <collision>
+            <origin xyz="0 0 0" rpy="0 0 0"/>
+            <geometry>
+                <mesh filename="package://manipulator_h_description/meshes/link_3.stl" scale="0.001 0.001 0.001"/>
+            </geometry>
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
Commit message: Addidtions to the model

File: manipulator_h_description/urdf/manipulator_h.xacro (robot description, xacro)
@@ -2,12 +2,34 @@
 <!-- Revolute-Revolute Manipulator -->
 <robot name="robotis_manipulator_h" xmlns:xacro="http://www.ros.org/wiki/xacro">
-    <!-- some parameters -->
-    <xacro:property name="pi" value="3.141592654" />
-    <!-- some parameters -->
-    <xacro:property name="pi" value="3.141592654" />
+<!--     <xacro:property name="pi" value="3.141592654" /> -->
     <!-- Import all Gazebo-customization elements, including Gazebo colors -->
     <xacro:include filename="$(find manipulator_h_description)/urdf/manipulator_h.gazebo" />
     <!-- Import Rviz colors -->
     <xacro:include filename="$(find manipulator_h_description)/urdf/materials.xacro" />
+<!--         IMPORT XTION_pro_live -->
+    <xacro:include filename="$(find manipulator_h_description)/urdf/xtion_pro_live.urdf.xacro"/>
+    <!-- Constants -->
+    <xacro:property name="deg_to_rad" value="0.01745329251994329577"/>
+    <xacro:property name="pi" value="3.141592654" />
+    <xacro:property name="M_SCALE" value="0.001 0.001 0.001"/>
+    <xacro:property name="M_PI" value="3.14159"/>
+    <xacro:macro name="inertial_matrix" params="mass">
+        <inertial>
+            <mass value="${mass}" />
+            <inertia ixx="1.0" ixy="0.0" ixz="0.0" iyy="0.5" iyz="0.0" izz="1.0" />
+        </inertial>
+    </xacro:macro>
+<!--    <xacro:macro name="transmission_block" params="joint_name">
+        <transmission name="tran1">
+            <type>transmission_interface/SimpleTransmission</type>
+            <joint name="${joint_name}">
+                <hardwareInterface>PositionJointInterface</hardwareInterface>
+            </joint>
+            <actuator name="motor1">
+                <hardwareInterface>PositionJointInterface</hardwareInterface>
+                <mechanicalReduction>1</mechanicalReduction>
+            </actuator>
+        </transmission>
+    </xacro:macro>-->
     <!-- Used for fixing robot to Gazebo 'link 1' -->
     <link name="world">
@@ -410,5 +432,5 @@
                 <mesh filename="package://manipulator_h_description/meshes/dist.stl" scale="1 1 1"/>
             </geometry>
-<!--             <material name="blue"/> -->
+            <!--             <material name="blue"/> -->
         </visual>
         <inertial>
@@ -421,4 +443,8 @@
         </inertial>
     </link>
+    <xacro:xtion_pro_live name="rgbd_camera" parent="end">
+        <origin xyz="0.05 0 -0.075" rpy="${180.0 * deg_to_rad} ${-10.0 * deg_to_rad} ${0 * deg_to_rad}"/>
+        <origin xyz="0.05 0 -0.075" rpy="${180.0 * deg_to_rad} ${-10.0 * deg_to_rad} ${0 * deg_to_rad}"/>
+    </xacro:xtion_pro_live>
     <!--     TRANSMISSIONS FOR THE GRIPPER -->
     <transmission name="joint_r1">
@@ -442,3 +468,8 @@
         </actuator>
     </transmission>
+     <gazebo>
+    <plugin name="gazebo_ros_control" filename="libgazebo_ros_control.so">
+    <robotNamespace>/robotis_manipulator_h</robotNamespace>
+    </plugin>
+    </gazebo>
 </robot>
